File: 299_RadioConfig/299_RadioConfig.kicad_pcb (KiCad board)
At the start: 2 copper layers, 0 parts

Commit message: Updated Radio Config, as ordered from JLCPCB
Parts:
- added BZ1: Buzzer, Buzzer_Beeper:Buzzer_TDK_PS1240P02BT_D12.2mm_H6.5mm, F.Cu at (191.0, 99.0)
- added C1: .1u, Capacitor_THT:C_Axial_L3.8mm_D2.6mm_P7.50mm_Horizontal, F.Cu at (144.8, 64.0)
- added C2: 470u, Capacitor_THT:C_Radial_D6.3mm_H11.0mm_P2.50mm, F.Cu at (155.0, 53.0)
- added C3: 470u, Capacitor_THT:C_Radial_D5.0mm_H11.0mm_P2.00mm, F.Cu at (148.0, 53.0)
- added C4: .1u, Capacitor_THT:C_Axial_L3.8mm_D2.6mm_P7.50mm_Horizontal, F.Cu at (132.0, 93.8)
- added DISP1: OLED Display, Connector_PinHeader_2.54mm:PinHeader_1x07_P2.54mm_Vertical, F.Cu at (154.0, 85.4)
- added LS1: Speaker, TerminalBlock_Phoenix:TerminalBlock_Phoenix_MKDS-1,5-2_1x02_P5.00mm_Horizontal, F.Cu at (137.0, 52.0)
- added R1: 2k, Resistor_THT:R_Axial_DIN0207_L6.3mm_D2.5mm_P10.16mm_Horizontal, F.Cu at (150.0, 64.9)
- added R2: 2k, Resistor_THT:R_Axial_DIN0207_L6.3mm_D2.5mm_P10.16mm_Horizontal, F.Cu at (155.0, 64.9)
- added R3: 10, Resistor_THT:R_Axial_DIN0207_L6.3mm_D2.5mm_P10.16mm_Horizontal, F.Cu at (144.9, 60.0)
- added SW1: Bourns PEC11R, Rotary_Encoder:RotaryEncoder_Alps_EC12E-Switch_Vertical_H20mm_CircularMountingHoles, F.Cu at (179.8, 55.5)
- added SW2: SW_Push, Connector_PinHeader_2.54mm:PinHeader_1x02_P2.54mm_Vertical, F.Cu at (182.0, 75.0)
- added SW3: SW_Push, Connector_PinHeader_2.54mm:PinHeader_1x02_P2.54mm_Vertical, F.Cu at (182.0, 68.0)
- added SW4: SW_Push, Connector_PinHeader_2.54mm:PinHeader_1x02_P2.54mm_Vertical, F.Cu at (182.0, 82.0)
- added SW5: SW_Push, Connector_PinHeader_2.54mm:PinHeader_1x02_P2.54mm_Vertical, F.Cu at (182.0, 89.0)
- added U1: RPi_Pico_TH, ECE:RPi_Pico_TH, B.Cu at (167.6, 79.0)
- added U2: RDA5807M_Module, ECE:RDA5807M_Module_TH, F.Cu at (142.0, 91.0)
- added U3: LM386, Package_DIP:DIP-8_W7.62mm, F.Cu at (137.2, 76.8)
Routing:
- net GND: track 0.00 -> 165.4 mm
- net Net-(DISP1-Pad2): track 0.00 -> 61.6 mm
- net Net-(U1-Pad11): track 0.00 -> 23.8 mm
- net Net-(C1-Pad1): track 0.00 -> 22.1 mm
- net Net-(R1-Pad2): track 0.00 -> 21.1 mm
- net Net-(SW1-PadS2): track 0.00 -> 19.6 mm
- net Net-(C4-Pad2): track 0.00 -> 17.3 mm
- net Net-(R2-Pad2): track 0.00 -> 16.9 mm
- net Net-(SW5-Pad1): track 0.00 -> 14.7 mm
- net Net-(C4-Pad1): track 0.00 -> 12.0 mm
- net Net-(DISP1-Pad6): track 0.00 -> 9.58 mm
- net Net-(DISP1-Pad5): track 0.00 -> 9.58 mm
- net Net-(C3-Pad2): track 0.00 -> 9.41 mm
- net Net-(C1-Pad2): track 0.00 -> 9.33 mm
- net Net-(SW4-Pad1): track 0.00 -> 9.05 mm
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- added copper zone on B.Cu, net GND
Other:
- board outline added: 75 x 65 mm
- board text added: "Simon - Aly ECE 299 Clock Radio"
